Commit message: move_base with odom root

File: simulator_ws/src/tb_gazebo_description/robots/kobuki_hexagons_kinect.urdf.xacro (robot description, xacro)
@@ -6,8 +6,14 @@
 -->
 <robot name="turtlebot" xmlns:xacro="http://ros.org/wiki/xacro">
+  <xacro:arg name="gpu" default="false"/>
+  <xacro:property name="gpu" value="$(arg gpu)" />
   <xacro:include filename="$(find tb_gazebo_description)/urdf/turtlebot_common_library.urdf.xacro" />
   <xacro:include filename="$(find tb_gazebo_description)/urdf/kobuki.urdf.xacro" />
   <xacro:include filename="$(find tb_gazebo_description)/urdf/stacks/hexagons.urdf.xacro"/>
   <xacro:include filename="$(find tb_gazebo_description)/urdf/sensors/kinect.urdf.xacro"/>
+  <xacro:include filename="$(find velodyne_description)/urdf/VLP-16.urdf.xacro"/>
+  <VLP-16 parent="base_link" name="velodyne" topic="/velodyne_points" hz="10" samples="440" gpu="${gpu}">
+    <origin xyz="0 0 0.4" rpy="0 0 0" />
+  </VLP-16>
   <kobuki/>
   <stack_hexagons parent="base_link"/>

Commit message: all modified

File: simulator_ws/src/tb_gazebo_description/robots/kobuki_hexagons_kinect.urdf.xacro (robot description, xacro)
@@ -10,4 +10,8 @@
   <xacro:include filename="$(find tb_gazebo_description)/urdf/stacks/hexagons.urdf.xacro"/>
   <xacro:include filename="$(find tb_gazebo_description)/urdf/sensors/kinect.urdf.xacro"/>
+  <xacro:include filename="$(find hector_sensors_description)/urdf/hokuyo_utm30lx.urdf.xacro" />
+  <xacro:hokuyo_utm30lx name="laser" parent="base_link" ros_topic="scan" update_rate="40" ray_count="1040" min_angle="180" max_angle="-180">
+    <origin xyz="0.00 0.00 0.20" rpy="0 0 0"/>
+  </xacro:hokuyo_utm30lx>
   <kobuki/>
   <stack_hexagons parent="base_link"/>

File: simulator_ws/src/tb_gazebo_description/urdf/turtlebot_properties.urdf.xacro (robot description, xacro)
@@ -19,5 +19,5 @@
      (currently in development and awaiting feedback)
    -->
-	<xacro:property name="cam_px" value="-0.087" />
+	<xacro:property name="cam_px" value="0.087" />
 <!--	<xacro:property name="cam_py" value="-0.0125" /> Y varies for different configurations. get sets in sensors_urdf -->
 	<xacro:property name="cam_pz" value="0.2870" />
